File: arduino_uno_shield.sch (EAGLE design)
At the start: 13 parts

Commit message: wiring up schematic
Parts:
- removed C1: (no value), SparkFun-Passives:CAPPTH
- removed C2: (no value), SparkFun-Passives:CAP_POLPTH2
- removed JP2, JP3, JP4, JP5: (no value), SparkFun-Connectors:M03PTH
- removed JP6: M02PTH, SparkFun-Connectors:M02PTH
- added C3: (no value), SparkFun-Passives:CAPPTH
- added C4: (no value), SparkFun-Passives:CAP_POLPTH2
- added MIC, POT1: (no value), SparkFun-Connectors:M03PTH
- added R2: (no value), SparkFun-Passives:RESISTORPTH-1/4W
Connections:
- new net 3.3V: MIC.3, POT1.3, U$2.VREF, U$3.VREFA
- new net 5V: U$2.VDD, U$3.VDD
- new net GND: C3.2, JP1.SLEEVE, MIC.1, POT1.1, R1.1, U$2.AGND, U$2.CH2, U$2.CH3, U$2.CH4, U$2.CH5, U$2.CH6, U$2.CH7, U$2.DGND
- new net N$1: MIC.2, U$2.CH0
- new net N$2: POT1.2, U$2.CH1
- new net N$3: R2.1, U$3.VOUTA
- new net N$4: U$1.D13, U$2.CLK, U$3.SCK
- new net N$8: C3.1, C4.+, R2.2
- new net N$9: C4.-, JP1.LEFT, JP1.RIGHT, R1.2
Other:
- moved on the sheet: JP1, R1, U$1, U$2, U$3

Commit message: wiring up schematic
Parts:
- removed C3: (no value), SparkFun-Passives:CAPPTH
- added C1: 0.1uF, SparkFun-Passives:CAPPTH
- added R3: 330, SparkFun-Passives:RESISTORPTH-1/4W
- C2: value (none) -> 10uF
- R1: value (none) -> 1.5K
- R2: value (none) -> 1K
- renumbered C4 to C2, JP1 to AUDIO_JACK
Connections:
- new net N$10: LED1.A, R3.1
- new net N$11: U$1.D8, U$3.~LDAC
- new net N$12: R3.2, U$1.*D6
- new net N$13: U$1.*D10, U$2.~CS/SHDN
- new net N$5: U$1.*D9, U$3.~CS
- new net N$6: U$1.D12, U$2.DOUT
- new net N$7: U$1.*D11, U$2.DIN, U$3.SDI
- net 5V: now also U$1.5V
- net GND: now also C1.2, LED1.C, R2.1, U$1.GND@0, U$1.GND@1, U$1.GND@2, U$3.AVSS; no longer C3.2, R1.1
- net N$3: now also R1.1; no longer R2.1
- net N$8: now also C1.1, R1.2; no longer C3.1, R2.2
- net N$9: now also R2.2; no longer R1.2
Other:
- moved on the sheet: LED1, R1, R2, U$1, U$2

Commit message: first attempt at board layout
Connections:
- net 3.3V: now also U$1.3.3V
Changed lines of the file:
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@@
 <pinref part="SUPPLY1" gate="G$1" pin="3.3V"/>
 <wire x1="-157.48" y1="66.04" x2="-157.48" y2="60.96" width="0.1524" layer="91"/>
-<wire x1="-157.48" y1="60.96" x2="-139.7" y2="60.96" width="0.1524" layer="91"/>
+<pinref part="U$1" gate="G$1" pin="3.3V"/>
+<wire x1="-157.48" y1="60.96" x2="-142.24" y2="60.96" width="0.1524" layer="91"/>
 </segment>
 </net>

Commit message: removed board
Parts:
- added POT2, POT3: (no value), SparkFun-Connectors:M03PTH
Connections:
- new net N$14: POT2.2, U$2.CH2
- new net N$15: POT3.2, U$2.CH3
- net 3.3V: now also POT2.3, POT3.3
- net GND: now also POT2.1, POT3.1; no longer U$2.CH2, U$2.CH3
Other:
- moved on the sheet: POT1, U$2

Commit message: re-created board
Parts:
- renumbered U$2 to MCP3208, U$3 to MCP4921
Changed lines of the file:
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@@
 <parts>
 <part name="U$1" library="SparkFun-Boards" deviceset="ARDUINO_R3_SHIELD" device=""/>
-<part name="U$2" library="Microchip_By_element14_Batch_1" deviceset="MCP3208-CI/P" device=""/>
-<part name="U$3" library="Microchip_By_element14_Batch_1" deviceset="MCP4921-E/P" device=""/>
+<part name="MCP3208" library="Microchip_By_element14_Batch_1" deviceset="MCP3208-CI/P" device=""/>
+<part name="MCP4921" library="Microchip_By_element14_Batch_1" deviceset="MCP4921-E/P" device=""/>
 <part name="GND1" library="SparkFun-Aesthetics" deviceset="GND" device=""/>
 <part name="R2" library="SparkFun-Passives" deviceset="RESISTOR" device="PTH-1/4W" value="1K"/>
@@
 <instances>
 <instance part="U$1" gate="G$1" x="-129.54" y="73.66"/>
-<instance part="U$2" gate="A" x="33.02" y="66.04"/>
-<instance part="U$3" gate="A" x="-101.6" y="2.54"/>
+<instance part="MCP3208" gate="A" x="33.02" y="66.04"/>
+<instance part="MCP4921" gate="A" x="-101.6" y="2.54"/>
 <instance part="GND1" gate="1" x="-68.58" y="-7.62"/>
 <instance part="R2" gate="G$1" x="-55.88" y="2.54" rot="R90"/>
@@
 </segment>
 <segment>
-<pinref part="U$3" gate="A" pin="AVSS"/>
+<pinref part="MCP4921" gate="A" pin="AVSS"/>
 <pinref part="GND8" gate="1" pin="GND"/>
 <wire x1="-119.38" y1="-10.16" x2="-121.92" y2="-10.16" width="0.1524" layer="91"/>
@@
 <pinref part="GND2" gate="1" pin="GND"/>
 <wire x1="12.7" y1="35.56" x2="12.7" y2="40.64" width="0.1524" layer="91"/>
-<pinref part="U$2" gate="A" pin="AGND"/>
+<pinref part="MCP3208" gate="A" pin="AGND"/>
 <wire x1="12.7" y1="40.64" x2="15.24" y2="40.64" width="0.1524" layer="91"/>
 <junction x="12.7" y="40.64"/>
 <wire x1="12.7" y1="40.64" x2="12.7" y2="43.18" width="0.1524" layer="91"/>
-<pinref part="U$2" gate="A" pin="DGND"/>
+<pinref part="MCP3208" gate="A" pin="DGND"/>
 <wire x1="12.7" y1="43.18" x2="15.24" y2="43.18" width="0.1524" layer="91"/>
 </segment>
@@
 <pinref part="GND12" gate="1" pin="GND"/>
 <wire x1="5.08" y1="35.56" x2="5.08" y2="48.26" width="0.1524" layer="91"/>
-<pinref part="U$2" gate="A" pin="CH7"/>
+<pinref part="MCP3208" gate="A" pin="CH7"/>
 <wire x1="5.08" y1="48.26" x2="15.24" y2="48.26" width="0.1524" layer="91"/>
 <junction x="5.08" y="48.26"/>
 <wire x1="5.08" y1="48.26" x2="5.08" y2="50.8" width="0.1524" layer="91"/>
-<pinref part="U$2" gate="A" pin="CH6"/>
+<pinref part="MCP3208" gate="A" pin="CH6"/>
 <wire x1="5.08" y1="50.8" x2="15.24" y2="50.8" width="0.1524" layer="91"/>
 <junction x="5.08" y="50.8"/>
 <wire x1="5.08" y1="50.8" x2="5.08" y2="53.34" width="0.1524" layer="91"/>
-<pinref part="U$2" gate="A" pin="CH5"/>
+<pinref part="MCP3208" gate="A" pin="CH5"/>
 <wire x1="5.08" y1="53.34" x2="15.24" y2="53.34" width="0.1524" layer="91"/>
 <junction x="5.08" y="53.34"/>
 <wire x1="5.08" y1="53.34" x2="5.08" y2="55.88" width="0.1524" layer="91"/>
-<pinref part="U$2" gate="A" pin="CH4"/>
+<pinref part="MCP3208" gate="A" pin="CH4"/>
 <wire x1="5.08" y1="55.88" x2="15.24" y2="55.88" width="0.1524" layer="91"/>
 </segment>
@@
 <pinref part="SUPPLY3" gate="G$1" pin="5V"/>
 <wire x1="12.7" y1="88.9" x2="12.7" y2="83.82" width="0.1524" layer="91"/>
-<pinref part="U$2" gate="A" pin="VDD"/>
+<pinref part="MCP3208" gate="A" pin="VDD"/>
 <wire x1="12.7" y1="83.82" x2="15.24" y2="83.82" width="0.1524" layer="91"/>
 </segment>
@@
 <pinref part="SUPPLY4" gate="G$1" pin="5V"/>
 <wire x1="-121.92" y1="15.24" x2="-121.92" y2="10.16" width="0.1524" layer="91"/>
-<pinref part="U$3" gate="A" pin="VDD"/>
+<pinref part="MCP4921" gate="A" pin="VDD"/>
 <wire x1="-121.92" y1="10.16" x2="-119.38" y2="10.16" width="0.1524" layer="91"/>
 </segment>
@@
 <pinref part="SUPPLY6" gate="G$1" pin="3.3V"/>
 <wire x1="5.08" y1="88.9" x2="5.08" y2="81.28" width="0.1524" layer="91"/>
-<pinref part="U$2" gate="A" pin="VREF"/>
+<pinref part="MCP3208" gate="A" pin="VREF"/>
 <wire x1="5.08" y1="81.28" x2="15.24" y2="81.28" width="0.1524" layer="91"/>
 </segment>
@@
 <pinref part="SUPPLY5" gate="G$1" pin="3.3V"/>
 <wire x1="-127" y1="15.24" x2="-127" y2="5.08" width="0.1524" layer="91"/>
-<pinref part="U$3" gate="A" pin="VREFA"/>
+<pinref part="MCP4921" gate="A" pin="VREFA"/>
 <wire x1="-127" y1="5.08" x2="-119.38" y2="5.08" width="0.1524" layer="91"/>
 </segment>
@@
 <net name="N$3" class="0">
 <segment>
-<pinref part="U$3" gate="A" pin="VOUTA"/>
+<pinref part="MCP4921" gate="A" pin="VOUTA"/>
 <pinref part="R1" gate="G$1" pin="1"/>
 <wire x1="-83.82" y1="10.16" x2="-81.28" y2="10.16" width="0.1524" layer="91"/>
@@
 <pinref part="U$1" gate="G$1" pin="D13"/>
 <wire x1="-116.84" y1="55.88" x2="-78.74" y2="55.88" width="0.1524" layer="91"/>
-<pinref part="U$2" gate="A" pin="CLK"/>
+<pinref part="MCP3208" gate="A" pin="CLK"/>
 <wire x1="15.24" y1="71.12" x2="-78.74" y2="71.12" width="0.1524" layer="91"/>
 <wire x1="-78.74" y1="71.12" x2="-78.74" y2="55.88" width="0.1524" layer="91"/>
 <junction x="-78.74" y="55.88"/>
-<pinref part="U$3" gate="A" pin="SCK"/>
+<pinref part="MCP4921" gate="A" pin="SCK"/>
 <wire x1="-119.38" y1="0" x2="-132.08" y2="0" width="0.1524" layer="91"/>
 <wire x1="-132.08" y1="0" x2="-132.08" y2="38.1" width="0.1524" layer="91"/>
@@
 <wire x1="-40.64" y1="55.88" x2="-35.56" y2="55.88" width="0.1524" layer="91"/>
 <wire x1="-35.56" y1="55.88" x2="-35.56" y2="66.04" width="0.1524" layer="91"/>
-<pinref part="U$2" gate="A" pin="CH0"/>
+<pinref part="MCP3208" gate="A" pin="CH0"/>
 <wire x1="-35.56" y1="66.04" x2="15.24" y2="66.04" width="0.1524" layer="91"/>
 </segment>
@@
 <wire x1="-40.64" y1="33.02" x2="-33.02" y2="33.02" width="0.1524" layer="91"/>
 <wire x1="-33.02" y1="33.02" x2="-33.02" y2="63.5" width="0.1524" layer="91"/>
-<pinref part="U$2" gate="A" pin="CH1"/>
+<pinref part="MCP3208" gate="A" pin="CH1"/>
 <wire x1="-33.02" y1="63.5" x2="15.24" y2="63.5" width="0.1524" layer="91"/>
 </segment>
@@
 <wire x1="-116.84" y1="58.42" x2="-81.28" y2="58.42" width="0.1524" layer="91"/>
 <junction x="-81.28" y="58.42"/>
-<pinref part="U$2" gate="A" pin="DOUT"/>
+<pinref part="MCP3208" gate="A" pin="DOUT"/>
 <wire x1="50.8" y1="83.82" x2="50.8" y2="96.52" width="0.1524" layer="91"/>
 <wire x1="50.8" y1="96.52" x2="-81.28" y2="96.52" width="0.1524" layer="91"/>
@@
 <wire x1="-116.84" y1="60.96" x2="-83.82" y2="60.96" width="0.1524" layer="91"/>
 <junction x="-83.82" y="60.96"/>
-<pinref part="U$2" gate="A" pin="DIN"/>
+<pinref part="MCP3208" gate="A" pin="DIN"/>
 <wire x1="15.24" y1="73.66" x2="-83.82" y2="73.66" width="0.1524" layer="91"/>
 <wire x1="-83.82" y1="73.66" x2="-83.82" y2="60.96" width="0.1524" layer="91"/>
@@
 <wire x1="-83.82" y1="40.64" x2="-134.62" y2="40.64" width="0.1524" layer="91"/>
 <wire x1="-134.62" y1="40.64" x2="-134.62" y2="-2.54" width="0.1524" layer="91"/>
-<pinref part="U$3" gate="A" pin="SDI"/>
+<pinref part="MCP4921" gate="A" pin="SDI"/>
 <wire x1="-134.62" y1="-2.54" x2="-119.38" y2="-2.54" width="0.1524" layer="91"/>
 </segment>
@@
 <wire x1="-99.06" y1="43.18" x2="-137.16" y2="43.18" width="0.1524" layer="91"/>
 <wire x1="-137.16" y1="43.18" x2="-137.16" y2="-5.08" width="0.1524" layer="91"/>
-<pinref part="U$3" gate="A" pin="~LDAC"/>
+<pinref part="MCP4921" gate="A" pin="~LDAC"/>
 <wire x1="-137.16" y1="-5.08" x2="-119.38" y2="-5.08" width="0.1524" layer="91"/>
 </segment>
@@
 <net name="N$13" class="0">
 <segment>
-<pinref part="U$2" gate="A" pin="~CS/SHDN"/>
+<pinref part="MCP3208" gate="A" pin="~CS/SHDN"/>
 <wire x1="15.24" y1="76.2" x2="-96.52" y2="76.2" width="0.1524" layer="91"/>
 <wire x1="-96.52" y1="76.2" x2="-96.52" y2="63.5" width="0.1524" layer="91"/>
@@
 <net name="N$5" class="0">
 <segment>
-<pinref part="U$3" gate="A" pin="~CS"/>
+<pinref part="MCP4921" gate="A" pin="~CS"/>
 <wire x1="-119.38" y1="2.54" x2="-129.54" y2="2.54" width="0.1524" layer="91"/>
 <wire x1="-129.54" y1="2.54" x2="-129.54" y2="35.56" width="0.1524" layer="91"/>
@@
 <wire x1="-15.24" y1="50.8" x2="-7.62" y2="50.8" width="0.1524" layer="91"/>
 <wire x1="-7.62" y1="50.8" x2="-7.62" y2="60.96" width="0.1524" layer="91"/>
-<pinref part="U$2" gate="A" pin="CH2"/>
+<pinref part="MCP3208" gate="A" pin="CH2"/>
 <wire x1="-7.62" y1="60.96" x2="15.24" y2="60.96" width="0.1524" layer="91"/>
 </segment>
@@
 <wire x1="-15.24" y1="27.94" x2="-5.08" y2="27.94" width="0.1524" layer="91"/>
 <wire x1="-5.08" y1="27.94" x2="-5.08" y2="58.42" width="0.1524" layer="91"/>
-<pinref part="U$2" gate="A" pin="CH3"/>
+<pinref part="MCP3208" gate="A" pin="CH3"/>
 <wire x1="-5.08" y1="58.42" x2="15.24" y2="58.42" width="0.1524" layer="91"/>
 </segment>

Commit message: save
Parts:
- renumbered MCP3208 to ADC, MCP4921 to DAC
Connections:
- net N$1 renamed AUD
Changed lines of the file:
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@@
 <parts>
 <part name="U$1" library="SparkFun-Boards" deviceset="ARDUINO_R3_SHIELD" device=""/>
-<part name="MCP3208" library="Microchip_By_element14_Batch_1" deviceset="MCP3208-CI/P" device=""/>
-<part name="MCP4921" library="Microchip_By_element14_Batch_1" deviceset="MCP4921-E/P" device=""/>
+<part name="ADC" library="Microchip_By_element14_Batch_1" deviceset="MCP3208-CI/P" device=""/>
+<part name="DAC" library="Microchip_By_element14_Batch_1" deviceset="MCP4921-E/P" device=""/>
 <part name="GND1" library="SparkFun-Aesthetics" deviceset="GND" device=""/>
 <part name="R2" library="SparkFun-Passives" deviceset="RESISTOR" device="PTH-1/4W" value="1K"/>
@@
 <instances>
 <instance part="U$1" gate="G$1" x="-129.54" y="73.66"/>
-<instance part="MCP3208" gate="A" x="33.02" y="66.04"/>
-<instance part="MCP4921" gate="A" x="-101.6" y="2.54"/>
+<instance part="ADC" gate="A" x="33.02" y="66.04"/>
+<instance part="DAC" gate="A" x="-101.6" y="2.54"/>
 <instance part="GND1" gate="1" x="-68.58" y="-7.62"/>
 <instance part="R2" gate="G$1" x="-55.88" y="2.54" rot="R90"/>
 <instance part="AUDIO_JACK" gate="G$1" x="-40.64" y="7.62" rot="R180"/>
-<instance part="MIC" gate="G$1" x="-48.26" y="55.88"/>
+<instance part="MIC" gate="G$1" x="-48.26" y="55.88" smashed="yes">
+<attribute name="VALUE" x="-50.8" y="48.26" size="1.778" layer="96"/>
+<attribute name="NAME" x="-50.8" y="61.722" size="1.778" layer="95"/>
+</instance>
 <instance part="POT1" gate="G$1" x="-48.26" y="33.02"/>
 <instance part="LED1" gate="G$1" x="-63.5" y="50.8"/>
@@
 </segment>
 <segment>
-<pinref part="MCP4921" gate="A" pin="AVSS"/>
+<pinref part="DAC" gate="A" pin="AVSS"/>
 <pinref part="GND8" gate="1" pin="GND"/>
 <wire x1="-119.38" y1="-10.16" x2="-121.92" y2="-10.16" width="0.1524" layer="91"/>
@@
 <pinref part="GND2" gate="1" pin="GND"/>
 <wire x1="12.7" y1="35.56" x2="12.7" y2="40.64" width="0.1524" layer="91"/>
-<pinref part="MCP3208" gate="A" pin="AGND"/>
+<pinref part="ADC" gate="A" pin="AGND"/>
 <wire x1="12.7" y1="40.64" x2="15.24" y2="40.64" width="0.1524" layer="91"/>
 <junction x="12.7" y="40.64"/>
 <wire x1="12.7" y1="40.64" x2="12.7" y2="43.18" width="0.1524" layer="91"/>
-<pinref part="MCP3208" gate="A" pin="DGND"/>
+<pinref part="ADC" gate="A" pin="DGND"/>
 <wire x1="12.7" y1="43.18" x2="15.24" y2="43.18" width="0.1524" layer="91"/>
 </segment>
@@
 <pinref part="GND12" gate="1" pin="GND"/>
 <wire x1="5.08" y1="35.56" x2="5.08" y2="48.26" width="0.1524" layer="91"/>
-<pinref part="MCP3208" gate="A" pin="CH7"/>
+<pinref part="ADC" gate="A" pin="CH7"/>
 <wire x1="5.08" y1="48.26" x2="15.24" y2="48.26" width="0.1524" layer="91"/>
 <junction x="5.08" y="48.26"/>
 <wire x1="5.08" y1="48.26" x2="5.08" y2="50.8" width="0.1524" layer="91"/>
-<pinref part="MCP3208" gate="A" pin="CH6"/>
+<pinref part="ADC" gate="A" pin="CH6"/>
 <wire x1="5.08" y1="50.8" x2="15.24" y2="50.8" width="0.1524" layer="91"/>
 <junction x="5.08" y="50.8"/>
 <wire x1="5.08" y1="50.8" x2="5.08" y2="53.34" width="0.1524" layer="91"/>
-<pinref part="MCP3208" gate="A" pin="CH5"/>
+<pinref part="ADC" gate="A" pin="CH5"/>
 <wire x1="5.08" y1="53.34" x2="15.24" y2="53.34" width="0.1524" layer="91"/>
 <junction x="5.08" y="53.34"/>
 <wire x1="5.08" y1="53.34" x2="5.08" y2="55.88" width="0.1524" layer="91"/>
-<pinref part="MCP3208" gate="A" pin="CH4"/>
+<pinref part="ADC" gate="A" pin="CH4"/>
 <wire x1="5.08" y1="55.88" x2="15.24" y2="55.88" width="0.1524" layer="91"/>
 </segment>
@@
 <pinref part="SUPPLY3" gate="G$1" pin="5V"/>
 <wire x1="12.7" y1="88.9" x2="12.7" y2="83.82" width="0.1524" layer="91"/>
-<pinref part="MCP3208" gate="A" pin="VDD"/>
+<pinref part="ADC" gate="A" pin="VDD"/>
 <wire x1="12.7" y1="83.82" x2="15.24" y2="83.82" width="0.1524" layer="91"/>
 </segment>
@@
 <pinref part="SUPPLY4" gate="G$1" pin="5V"/>
 <wire x1="-121.92" y1="15.24" x2="-121.92" y2="10.16" width="0.1524" layer="91"/>
-<pinref part="MCP4921" gate="A" pin="VDD"/>
+<pinref part="DAC" gate="A" pin="VDD"/>
 <wire x1="-121.92" y1="10.16" x2="-119.38" y2="10.16" width="0.1524" layer="91"/>
 </segment>
@@
 <pinref part="SUPPLY6" gate="G$1" pin="3.3V"/>
 <wire x1="5.08" y1="88.9" x2="5.08" y2="81.28" width="0.1524" layer="91"/>
-<pinref part="MCP3208" gate="A" pin="VREF"/>
+<pinref part="ADC" gate="A" pin="VREF"/>
 <wire x1="5.08" y1="81.28" x2="15.24" y2="81.28" width="0.1524" layer="91"/>
 </segment>
@@
 <pinref part="SUPPLY5" gate="G$1" pin="3.3V"/>
 <wire x1="-127" y1="15.24" x2="-127" y2="5.08" width="0.1524" layer="91"/>
-<pinref part="MCP4921" gate="A" pin="VREFA"/>
+<pinref part="DAC" gate="A" pin="VREFA"/>
 <wire x1="-127" y1="5.08" x2="-119.38" y2="5.08" width="0.1524" layer="91"/>
 </segment>
@@
 <net name="N$3" class="0">
 <segment>
-<pinref part="MCP4921" gate="A" pin="VOUTA"/>
+<pinref part="DAC" gate="A" pin="VOUTA"/>
 <pinref part="R1" gate="G$1" pin="1"/>
 <wire x1="-83.82" y1="10.16" x2="-81.28" y2="10.16" width="0.1524" layer="91"/>
@@
 <pinref part="U$1" gate="G$1" pin="D13"/>
 <wire x1="-116.84" y1="55.88" x2="-78.74" y2="55.88" width="0.1524" layer="91"/>
-<pinref part="MCP3208" gate="A" pin="CLK"/>
+<pinref part="ADC" gate="A" pin="CLK"/>
 <wire x1="15.24" y1="71.12" x2="-78.74" y2="71.12" width="0.1524" layer="91"/>
 <wire x1="-78.74" y1="71.12" x2="-78.74" y2="55.88" width="0.1524" layer="91"/>
 <junction x="-78.74" y="55.88"/>
-<pinref part="MCP4921" gate="A" pin="SCK"/>
+<pinref part="DAC" gate="A" pin="SCK"/>
 <wire x1="-119.38" y1="0" x2="-132.08" y2="0" width="0.1524" layer="91"/>
 <wire x1="-132.08" y1="0" x2="-132.08" y2="38.1" width="0.1524" layer="91"/>
@@
 </segment>
 </net>
-<net name="N$1" class="0">
+<net name="AUD" class="0">
 <segment>
 <pinref part="MIC" gate="G$1" pin="2"/>
 <wire x1="-40.64" y1="55.88" x2="-35.56" y2="55.88" width="0.1524" layer="91"/>
 <wire x1="-35.56" y1="55.88" x2="-35.56" y2="66.04" width="0.1524" layer="91"/>
-<pinref part="MCP3208" gate="A" pin="CH0"/>
+<pinref part="ADC" gate="A" pin="CH0"/>
 <wire x1="-35.56" y1="66.04" x2="15.24" y2="66.04" width="0.1524" layer="91"/>
 </segment>
@@
 <wire x1="-40.64" y1="33.02" x2="-33.02" y2="33.02" width="0.1524" layer="91"/>
 <wire x1="-33.02" y1="33.02" x2="-33.02" y2="63.5" width="0.1524" layer="91"/>
-<pinref part="MCP3208" gate="A" pin="CH1"/>
+<pinref part="ADC" gate="A" pin="CH1"/>
 <wire x1="-33.02" y1="63.5" x2="15.24" y2="63.5" width="0.1524" layer="91"/>
 </segment>
@@
 <wire x1="-116.84" y1="58.42" x2="-81.28" y2="58.42" width="0.1524" layer="91"/>
 <junction x="-81.28" y="58.42"/>
-<pinref part="MCP3208" gate="A" pin="DOUT"/>
+<pinref part="ADC" gate="A" pin="DOUT"/>
 <wire x1="50.8" y1="83.82" x2="50.8" y2="96.52" width="0.1524" layer="91"/>
 <wire x1="50.8" y1="96.52" x2="-81.28" y2="96.52" width="0.1524" layer="91"/>
@@
 <wire x1="-116.84" y1="60.96" x2="-83.82" y2="60.96" width="0.1524" layer="91"/>
 <junction x="-83.82" y="60.96"/>
-<pinref part="MCP3208" gate="A" pin="DIN"/>
+<pinref part="ADC" gate="A" pin="DIN"/>
 <wire x1="15.24" y1="73.66" x2="-83.82" y2="73.66" width="0.1524" layer="91"/>
 <wire x1="-83.82" y1="73.66" x2="-83.82" y2="60.96" width="0.1524" layer="91"/>
@@
 <wire x1="-83.82" y1="40.64" x2="-134.62" y2="40.64" width="0.1524" layer="91"/>
 <wire x1="-134.62" y1="40.64" x2="-134.62" y2="-2.54" width="0.1524" layer="91"/>
-<pinref part="MCP4921" gate="A" pin="SDI"/>
+<pinref part="DAC" gate="A" pin="SDI"/>
 <wire x1="-134.62" y1="-2.54" x2="-119.38" y2="-2.54" width="0.1524" layer="91"/>
 </segment>
@@
 <wire x1="-99.06" y1="43.18" x2="-137.16" y2="43.18" width="0.1524" layer="91"/>
 <wire x1="-137.16" y1="43.18" x2="-137.16" y2="-5.08" width="0.1524" layer="91"/>
-<pinref part="MCP4921" gate="A" pin="~LDAC"/>
+<pinref part="DAC" gate="A" pin="~LDAC"/>
 <wire x1="-137.16" y1="-5.08" x2="-119.38" y2="-5.08" width="0.1524" layer="91"/>
 </segment>
@@
 <net name="N$13" class="0">
 <segment>
-<pinref part="MCP3208" gate="A" pin="~CS/SHDN"/>
+<pinref part="ADC" gate="A" pin="~CS/SHDN"/>
 <wire x1="15.24" y1="76.2" x2="-96.52" y2="76.2" width="0.1524" layer="91"/>
 <wire x1="-96.52" y1="76.2" x2="-96.52" y2="63.5" width="0.1524" layer="91"/>
@@
 <net name="N$5" class="0">
 <segment>
-<pinref part="MCP4921" gate="A" pin="~CS"/>
+<pinref part="DAC" gate="A" pin="~CS"/>
 <wire x1="-119.38" y1="2.54" x2="-129.54" y2="2.54" width="0.1524" layer="91"/>
 <wire x1="-129.54" y1="2.54" x2="-129.54" y2="35.56" width="0.1524" layer="91"/>
@@
 <wire x1="-15.24" y1="50.8" x2="-7.62" y2="50.8" width="0.1524" layer="91"/>
 <wire x1="-7.62" y1="50.8" x2="-7.62" y2="60.96" width="0.1524" layer="91"/>
-<pinref part="MCP3208" gate="A" pin="CH2"/>
+<pinref part="ADC" gate="A" pin="CH2"/>
 <wire x1="-7.62" y1="60.96" x2="15.24" y2="60.96" width="0.1524" layer="91"/>
 </segment>
@@
 <wire x1="-15.24" y1="27.94" x2="-5.08" y2="27.94" width="0.1524" layer="91"/>
 <wire x1="-5.08" y1="27.94" x2="-5.08" y2="58.42" width="0.1524" layer="91"/>
-<pinref part="MCP3208" gate="A" pin="CH3"/>
+<pinref part="ADC" gate="A" pin="CH3"/>
 <wire x1="-5.08" y1="58.42" x2="15.24" y2="58.42" width="0.1524" layer="91"/>
 </segment>
