File: arduino_uno_shield.brd (EAGLE design)
At the start: 53 x 57.1 mm, 20 parts

Commit message: refining board layout to remove via:
Routing:
- net GND: track 206.4 -> 0.00 mm
- net 3.3V: track 88.0 -> 0.00 mm
- net N$12: track 53.7 -> 0.00 mm, vias 1 -> 0
- net 5V: track 45.7 -> 0.00 mm
- net SPI_MOSI: track 45.1 -> 0.00 mm
- net N$18: track 34.5 -> 0.00 mm
- net N$17: track 33.6 -> 0.00 mm
- net N$1: track 31.9 -> 0.00 mm
- net N$9: track 29.1 -> 0.00 mm
- net SPI_CLK: track 27.0 -> 0.00 mm
- net AUD: track 23.8 -> 0.00 mm
- net N$16: track 23.5 -> 0.00 mm
- net SPI_MISO: track 22.3 -> 0.00 mm
- net N$11: track 22.2 -> 0.00 mm
- net CS_ADC: track 22.2 -> 0.00 mm
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
Commit message: saving work, this version ordered
Parts:
- moved LED 36.9 mm to (14.0, 62.2)
- moved R3 34.3 mm to (14.0, 68.6)
- moved MCP3208 14.0 mm to (10.2, 55.9)
- moved MCP4921 12.7 mm to (17.8, 26.7)
- moved C1 9.25 mm to (33.0, 34.3)
- moved R2 8.03 mm to (27.9, 39.4), turned to 0 degrees
- moved R1 4.58 mm to (27.9, 44.5), turned to 0 degrees
- moved C2 2.54 mm to (39.4, 41.9), turned to 90 degrees
Routing:
- net GND: track 0.00 -> 204.1 mm
- net 3.3V: track 0.00 -> 97.2 mm
- net N$12: track 0.00 -> 62.3 mm
- net 5V: track 0.00 -> 50.5 mm
- net N$1: track 0.00 -> 36.8 mm
- net AUD: track 0.00 -> 35.7 mm
- net N$16: track 0.00 -> 34.9 mm
- net N$11: track 0.00 -> 33.5 mm
- net CS_DAC: track 0.00 -> 33.3 mm
- net N$2: track 0.00 -> 32.1 mm
- net SPI_MOSI: track 0.00 -> 32.0 mm
- net N$9: track 0.00 -> 29.3 mm
- net N$17: track 0.00 -> 28.3 mm
- net N$18: track 0.00 -> 23.9 mm
- net SPI_CLK: track 0.00 -> 23.7 mm
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Other:
- board text added: "Ultimate Voice Changer Shield v1.0.1"
- board text removed: "Ultimate Voice Changer Shield v1.0.0"
