File: eagle_schematics/arduino_shield_v2/arduino_uno_shield.sch (EAGLE design)
At the start: 15 parts, among them IC1 TL072P

Commit message: Save
Parts:
- IC1: value TL072P -> TLV2462CP
- renumbered R3 to R2
Changed lines of the file:
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@@
 <?xml version="1.0" encoding="utf-8"?>
 <!DOCTYPE eagle SYSTEM "eagle.dtd">
-<eagle version="7.5.0">
+<eagle version="7.1.0">
 <drawing>
 <settings>
@@
 <part name="GND7" library="SparkFun-Aesthetics" deviceset="GND" device=""/>
 <part name="GND8" library="SparkFun-Aesthetics" deviceset="GND" device=""/>
-<part name="R3" library="SparkFun-Passives" deviceset="RESISTOR" device="PTH-1/4W" value="330"/>
+<part name="R2" library="SparkFun-Passives" deviceset="RESISTOR" device="PTH-1/4W" value="330"/>
 <part name="SUPPLY1" library="SparkFun-Aesthetics" deviceset="3.3V" device=""/>
 <part name="SUPPLY9" library="SparkFun-Aesthetics" deviceset="5V" device=""/>
@@
 <part name="GND14" library="SparkFun-Aesthetics" deviceset="GND" device=""/>
 <part name="EXT_LED" library="SparkFun-Connectors" deviceset="M02" device="3.5MM"/>
-<part name="IC1" library="linear" deviceset="TL072" device="P"/>
+<part name="IC1" library="linear" deviceset="TL072" device="P" value="TLV2462CP"/>
 <part name="SUPPLY15" library="SparkFun-Aesthetics" deviceset="5V" device=""/>
 <part name="C2" library="SparkFun-Capacitors" deviceset="CAP_POL" device="PTH1" value="100uF"/>
@@
 <instance part="GND7" gate="1" x="-48.26" y="-7.62"/>
 <instance part="GND8" gate="1" x="-121.92" y="-17.78"/>
-<instance part="R3" gate="G$1" x="-63.5" y="58.42" rot="R90"/>
+<instance part="R2" gate="G$1" x="-63.5" y="58.42" rot="R90"/>
 <instance part="SUPPLY1" gate="G$1" x="-157.48" y="66.04"/>
 <instance part="SUPPLY9" gate="G$1" x="-149.86" y="76.2"/>
@@
 <segment>
 <pinref part="LED" gate="G$1" pin="A"/>
-<pinref part="R3" gate="G$1" pin="1"/>
+<pinref part="R2" gate="G$1" pin="1"/>
 </segment>
 </net>
@@
 <wire x1="-91.44" y1="73.66" x2="-91.44" y2="66.04" width="0.1524" layer="91"/>
 <wire x1="-91.44" y1="66.04" x2="-63.5" y2="66.04" width="0.1524" layer="91"/>
-<pinref part="R3" gate="G$1" pin="2"/>
+<pinref part="R2" gate="G$1" pin="2"/>
 <wire x1="-63.5" y1="66.04" x2="-63.5" y2="63.5" width="0.1524" layer="91"/>
 <pinref part="EXT_LED" gate="G$1" pin="1"/>
