File: eagle_schematics/arduino_shield/v110.sch (EAGLE design)
At the start: 10 parts, among them U1 ARDUINO_SHIELDLABEL

Commit message: new board rev
Parts:
- added ADC2, ADC3, ADC4: TRIMPOT-PTH-KNOB, SparkFun-Electromechanical:TRIMPOT-PTH-KNOB
- added EXT_LED: M02LOCK, SparkFun-Connectors:M02LOCK
- added MIC: (no value), SparkFun-Connectors:M03LOCK
- added R4: (no value), SparkFun-Resistors:1KOHM-1/4W-5%(PTH)
- C1: value (none) -> 0.1uF
- C2: value (none) -> 10uF
- R1: value (none) -> 330
- R2: value (none) -> 1.5k
- R3: value (none) -> 1k
Connections:
- new net N$5: EXT_LED.1, R4.2
- net 3.3V: now also ADC2.CCW, ADC3.CCW, ADC4.CCW, MIC.3
- net ADC1: now also MIC.1
- net ADC2: now also ADC2.WIPER
- net ADC3: now also ADC3.WIPER
- net ADC4: now also ADC4.WIPER
- net GND: now also ADC2.CW, ADC3.CW, ADC4.CW, EXT_LED.2, MIC.2
- net LED: now also R4.1, U1.*D6
Changed lines of the file:
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@@
 <part name="U$1" library="Microchip_By_element14_Batch_1" deviceset="MCP4921-E/P" device=""/>
 <part name="U$2" library="Microchip_By_element14_Batch_1" deviceset="MCP3204-CI/P" device=""/>
-<part name="R1" library="SparkFun-Resistors" deviceset="1KOHM-1/4W-5%(PTH)" device=""/>
-<part name="R2" library="SparkFun-Resistors" deviceset="1KOHM-1/4W-5%(PTH)" device=""/>
-<part name="R3" library="SparkFun-Resistors" deviceset="1KOHM-1/4W-5%(PTH)" device=""/>
+<part name="R1" library="SparkFun-Resistors" deviceset="1KOHM-1/4W-5%(PTH)" device="" value="330"/>
+<part name="R2" library="SparkFun-Resistors" deviceset="1KOHM-1/4W-5%(PTH)" device="" value="1.5k"/>
+<part name="R3" library="SparkFun-Resistors" deviceset="1KOHM-1/4W-5%(PTH)" device="" value="1k"/>
 <part name="LED1" library="SparkFun-LED" deviceset="LED" device="5MM"/>
-<part name="C1" library="SparkFun-Capacitors" deviceset="CAP" device="PTH1"/>
-<part name="C2" library="SparkFun-Capacitors" deviceset="CAP_POL" device="PTH2"/>
+<part name="C1" library="SparkFun-Capacitors" deviceset="CAP" device="PTH1" value="0.1uF"/>
+<part name="C2" library="SparkFun-Capacitors" deviceset="CAP_POL" device="PTH2" value="10uF"/>
 <part name="GND1" library="SparkFun-Aesthetics" deviceset="GND" device=""/>
 <part name="GND2" library="SparkFun-Aesthetics" deviceset="GND" device=""/>
 <part name="JP1" library="SparkFun-Connectors" deviceset="AUDIO-JACK" device="PTH"/>
 <part name="GND3" library="SparkFun-Aesthetics" deviceset="GND" device=""/>
+<part name="MIC" library="SparkFun-Connectors" deviceset="M03" device="LOCK"/>
+<part name="EXT_LED" library="SparkFun-Connectors" deviceset="M02" device="LOCK"/>
+<part name="R4" library="SparkFun-Resistors" deviceset="1KOHM-1/4W-5%(PTH)" device=""/>
+<part name="ADC2" library="SparkFun-Electromechanical" deviceset="TRIMPOT" device="-PTH-KNOB"/>
+<part name="ADC3" library="SparkFun-Electromechanical" deviceset="TRIMPOT" device="-PTH-KNOB"/>
+<part name="ADC4" library="SparkFun-Electromechanical" deviceset="TRIMPOT" device="-PTH-KNOB"/>
 </parts>
 <sheets>
@@
 <instance part="JP1" gate="G$1" x="142.24" y="83.82" rot="R180"/>
 <instance part="GND3" gate="1" x="134.62" y="66.04"/>
+<instance part="MIC" gate="G$1" x="-5.08" y="15.24"/>
+<instance part="EXT_LED" gate="G$1" x="40.64" y="17.78" rot="R180"/>
+<instance part="R4" gate="G$1" x="25.4" y="17.78"/>
+<instance part="ADC2" gate="R?" x="-5.08" y="-7.62"/>
+<instance part="ADC3" gate="R?" x="-5.08" y="-27.94"/>
+<instance part="ADC4" gate="R?" x="38.1" y="-27.94"/>
 </instances>
 <busses>
@@
 <wire x1="134.62" y1="81.28" x2="134.62" y2="68.58" width="0.1524" layer="91"/>
 </segment>
+<segment>
+<pinref part="MIC" gate="G$1" pin="2"/>
+<wire x1="2.54" y1="15.24" x2="10.16" y2="15.24" width="0.1524" layer="91"/>
+<label x="2.54" y="15.24" size="1.778" layer="95"/>
+</segment>
+<segment>
+<pinref part="EXT_LED" gate="G$1" pin="2"/>
+<wire x1="33.02" y1="15.24" x2="27.94" y2="15.24" width="0.1524" layer="91"/>
+<label x="27.94" y="15.24" size="1.778" layer="95"/>
+</segment>
+<segment>
+<pinref part="ADC2" gate="R?" pin="CW"/>
+<wire x1="0" y1="-7.62" x2="7.62" y2="-7.62" width="0.1524" layer="91"/>
+<label x="0" y="-7.62" size="1.778" layer="95"/>
+</segment>
+<segment>
+<pinref part="ADC3" gate="R?" pin="CW"/>
+<wire x1="0" y1="-27.94" x2="7.62" y2="-27.94" width="0.1524" layer="91"/>
+<label x="2.54" y="-27.94" size="1.778" layer="95"/>
+</segment>
+<segment>
+<pinref part="ADC4" gate="R?" pin="CW"/>
+<wire x1="43.18" y1="-27.94" x2="53.34" y2="-27.94" width="0.1524" layer="91"/>
+<label x="45.72" y="-27.94" size="1.778" layer="95"/>
+</segment>
 </net>
 <net name="LED" class="0">
@@
 <label x="-7.62" y="33.02" size="1.778" layer="95"/>
 </segment>
+<segment>
+<pinref part="U1" gate="G$1" pin="*D6"/>
+<wire x1="20.32" y1="71.12" x2="27.94" y2="71.12" width="0.1524" layer="91"/>
+<label x="20.32" y="71.12" size="1.778" layer="95"/>
+</segment>
+<segment>
+<pinref part="R4" gate="G$1" pin="1"/>
+<wire x1="20.32" y1="17.78" x2="12.7" y2="17.78" width="0.1524" layer="91"/>
+<label x="12.7" y="17.78" size="1.778" layer="95"/>
+</segment>
 </net>
 <net name="SCK" class="0">
@@
 <label x="53.34" y="81.28" size="1.778" layer="95"/>
 </segment>
+<segment>
+<pinref part="MIC" gate="G$1" pin="3"/>
+<wire x1="2.54" y1="17.78" x2="10.16" y2="17.78" width="0.1524" layer="91"/>
+<label x="2.54" y="17.78" size="1.778" layer="95"/>
+</segment>
+<segment>
+<pinref part="ADC2" gate="R?" pin="CCW"/>
+<wire x1="-10.16" y1="-7.62" x2="-17.78" y2="-7.62" width="0.1524" layer="91"/>
+<label x="-17.78" y="-7.62" size="1.778" layer="95"/>
+</segment>
+<segment>
+<pinref part="ADC3" gate="R?" pin="CCW"/>
+<wire x1="-10.16" y1="-27.94" x2="-17.78" y2="-27.94" width="0.1524" layer="91"/>
+<label x="-17.78" y="-27.94" size="1.778" layer="95"/>
+</segment>
+<segment>
+<pinref part="ADC4" gate="R?" pin="CCW"/>
+<wire x1="33.02" y1="-27.94" x2="22.86" y2="-27.94" width="0.1524" layer="91"/>
+<label x="22.86" y="-27.94" size="1.778" layer="95"/>
+</segment>
 </net>
 <net name="ADC1" class="0">
@@
 <label x="50.8" y="15.24" size="1.778" layer="95"/>
 </segment>
+<segment>
+<pinref part="MIC" gate="G$1" pin="1"/>
+<wire x1="2.54" y1="12.7" x2="10.16" y2="12.7" width="0.1524" layer="91"/>
+<label x="2.54" y="12.7" size="1.778" layer="95"/>
+</segment>
 </net>
 <net name="ADC2" class="0">
@@
 <label x="50.8" y="12.7" size="1.778" layer="95"/>
 </segment>
+<segment>
+<pinref part="ADC2" gate="R?" pin="WIPER"/>
+<wire x1="-5.08" y1="-2.54" x2="-5.08" y2="5.08" width="0.1524" layer="91"/>
+<label x="-5.08" y="-2.54" size="1.778" layer="95"/>
+</segment>
 </net>
 <net name="ADC3" class="0">
@@
 <label x="50.8" y="10.16" size="1.778" layer="95"/>
 </segment>
+<segment>
+<pinref part="ADC3" gate="R?" pin="WIPER"/>
+<wire x1="-5.08" y1="-22.86" x2="-5.08" y2="-15.24" width="0.1524" layer="91"/>
+<label x="-5.08" y="-22.86" size="1.778" layer="95"/>
+</segment>
 </net>
 <net name="ADC4" class="0">
@@
 <wire x1="58.42" y1="7.62" x2="50.8" y2="7.62" width="0.1524" layer="91"/>
 <label x="50.8" y="7.62" size="1.778" layer="95"/>
+</segment>
+<segment>
+<pinref part="ADC4" gate="R?" pin="WIPER"/>
+<wire x1="38.1" y1="-22.86" x2="38.1" y2="-15.24" width="0.1524" layer="91"/>
+<label x="38.1" y="-22.86" size="1.778" layer="95"/>
 </segment>
 </net>
@@
 </segment>
 </net>
+<net name="N$5" class="0">
+<segment>
+<pinref part="R4" gate="G$1" pin="2"/>
+<pinref part="EXT_LED" gate="G$1" pin="1"/>
+<wire x1="30.48" y1="17.78" x2="33.02" y2="17.78" width="0.1524" layer="91"/>
+</segment>
+</net>
 </nets>
 </sheet>
 </sheets>
+<errors>
+</errors>
 </schematic>
 </drawing>

Commit message: clean up board
Parts:
- renumbered LED1 to LED
Changed lines of the file:
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@@
 <part name="R2" library="SparkFun-Resistors" deviceset="1KOHM-1/4W-5%(PTH)" device="" value="1.5k"/>
 <part name="R3" library="SparkFun-Resistors" deviceset="1KOHM-1/4W-5%(PTH)" device="" value="1k"/>
-<part name="LED1" library="SparkFun-LED" deviceset="LED" device="5MM"/>
+<part name="LED" library="SparkFun-LED" deviceset="LED" device="5MM"/>
 <part name="C1" library="SparkFun-Capacitors" deviceset="CAP" device="PTH1" value="0.1uF"/>
 <part name="C2" library="SparkFun-Capacitors" deviceset="CAP_POL" device="PTH2" value="10uF"/>
@@
 <instance part="R2" gate="G$1" x="104.14" y="86.36"/>
 <instance part="R3" gate="G$1" x="124.46" y="78.74" rot="R90"/>
-<instance part="LED1" gate="G$1" x="17.78" y="33.02" rot="R90"/>
+<instance part="LED" gate="G$1" x="17.78" y="33.02" rot="R90"/>
 <instance part="C1" gate="G$1" x="111.76" y="78.74"/>
 <instance part="C2" gate="G$1" x="116.84" y="86.36" rot="R90"/>
@@
 <segment>
 <pinref part="R1" gate="G$1" pin="2"/>
-<pinref part="LED1" gate="G$1" pin="A"/>
+<pinref part="LED" gate="G$1" pin="A"/>
 <wire x1="10.16" y1="33.02" x2="15.24" y2="33.02" width="0.1524" layer="91"/>
 </segment>
@@
 <net name="GND" class="0">
 <segment>
-<pinref part="LED1" gate="G$1" pin="C"/>
+<pinref part="LED" gate="G$1" pin="C"/>
 <wire x1="22.86" y1="33.02" x2="27.94" y2="33.02" width="0.1524" layer="91"/>
 <label x="27.94" y="33.02" size="1.778" layer="95"/>

Commit message: clean up board
Parts:
- renumbered MIC to ADC1_MIC
Changed lines of the file:
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@@
 <part name="JP1" library="SparkFun-Connectors" deviceset="AUDIO-JACK" device="PTH"/>
 <part name="GND3" library="SparkFun-Aesthetics" deviceset="GND" device=""/>
-<part name="MIC" library="SparkFun-Connectors" deviceset="M03" device="LOCK"/>
+<part name="ADC1_MIC" library="SparkFun-Connectors" deviceset="M03" device="LOCK"/>
 <part name="EXT_LED" library="SparkFun-Connectors" deviceset="M02" device="LOCK"/>
 <part name="R4" library="SparkFun-Resistors" deviceset="1KOHM-1/4W-5%(PTH)" device=""/>
@@
 <instance part="JP1" gate="G$1" x="142.24" y="83.82" rot="R180"/>
 <instance part="GND3" gate="1" x="134.62" y="66.04"/>
-<instance part="MIC" gate="G$1" x="-5.08" y="15.24"/>
+<instance part="ADC1_MIC" gate="G$1" x="-5.08" y="15.24"/>
 <instance part="EXT_LED" gate="G$1" x="40.64" y="17.78" rot="R180"/>
 <instance part="R4" gate="G$1" x="25.4" y="17.78"/>
@@
 </segment>
 <segment>
-<pinref part="MIC" gate="G$1" pin="2"/>
+<pinref part="ADC1_MIC" gate="G$1" pin="2"/>
 <wire x1="2.54" y1="15.24" x2="10.16" y2="15.24" width="0.1524" layer="91"/>
 <label x="2.54" y="15.24" size="1.778" layer="95"/>
@@
 </segment>
 <segment>
-<pinref part="MIC" gate="G$1" pin="3"/>
+<pinref part="ADC1_MIC" gate="G$1" pin="3"/>
 <wire x1="2.54" y1="17.78" x2="10.16" y2="17.78" width="0.1524" layer="91"/>
 <label x="2.54" y="17.78" size="1.778" layer="95"/>
@@
 </segment>
 <segment>
-<pinref part="MIC" gate="G$1" pin="1"/>
+<pinref part="ADC1_MIC" gate="G$1" pin="1"/>
 <wire x1="2.54" y1="12.7" x2="10.16" y2="12.7" width="0.1524" layer="91"/>
 <label x="2.54" y="12.7" size="1.778" layer="95"/>
