File: eagle_schematics/arduino_shield/v110.brd (EAGLE design)
At the start: 100 x 80 mm, 10 parts, among them U1 ARDUINO_SHIELDLABEL

Commit message: new board rev
Parts:
- added ADC2, ADC3, ADC4: TRIMPOT-PTH-KNOB, SparkFun-Electromechanical:3386U
- added EXT_LED: M02LOCK, SparkFun-Connectors:1X02_LOCK
- added MIC: (no value), SparkFun-Connectors:1X03_LOCK
- added R4: (no value), SparkFun-Resistors:AXIAL-0.3
- C1: value (none) -> 0.1uF
- C2: value (none) -> 10uF
- R1: value (none) -> 330
- R2: value (none) -> 1.5k
- R3: value (none) -> 1k
- moved R3 21.7 mm to (29.2, 29.2)
- moved LED1 17.3 mm to (16.5, 62.2), turned to 90 degrees
- moved C1 12.5 mm to (38.1, 25.4), turned to 270 degrees
- moved C2 9.16 mm to (52.1, 34.3)
- moved U$2 8.89 mm to (12.7, 54.6)
- moved R2 7.73 mm to (29.2, 33.0)
- moved JP1 7.18 mm to (48.3, 21.6), turned to 90 degrees
- moved U$1 6.35 mm to (20.3, 26.7)
- moved R1 6.35 mm to (16.5, 67.3)
Connections:
- new net N$5: EXT_LED.1, R4.P$2
- net 3.3V: now also ADC2.1, ADC3.1, ADC4.1, MIC.3
- net ADC1: now also MIC.1
- net ADC2: now also ADC2.2
- net ADC3: now also ADC3.2
- net ADC4: now also ADC4.2
- net GND: now also ADC2.3, ADC3.3, ADC4.3, EXT_LED.2, MIC.2
- net LED: now also R4.P$1, U1.D6
Routing:
- net GND: track 0.00 -> 131.9 mm
- net 3.3V: track 0.00 -> 90.3 mm
- net LED: track 0.00 -> 51.0 mm
- net 5V: track 0.00 -> 50.3 mm
- net ADC2: track 0.00 -> 39.5 mm
- net ADC3: track 0.00 -> 31.6 mm
- net MOSI: track 0.00 -> 30.7 mm
- net CS_DAC: track 0.00 -> 30.1 mm
- net LDAC: track 0.00 -> 30.0 mm
- net N$4: track 0.00 -> 27.9 mm
- net ADC4: track 0.00 -> 24.5 mm
- net N$3: track 0.00 -> 24.4 mm
- net SCK: track 0.00 -> 23.1 mm
- net ADC1: track 0.00 -> 18.0 mm
- net CS_ADC: track 0.00 -> 11.5 mm
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Other:
- board size 100 x 80 mm -> 54.3 x 59.7 mm
- board text added: "3.3V"
- board text added: "ADC1"
- board text added: "GND"
- board text added: "MCP3204"
- board text added: "MCP4921"
- board text added: "SuperAwesomeRobots.com"
- board text added: "Ultimate Voice Changer 1.1"

Commit message: clean up board
Parts:
- renumbered LED1 to LED
Changed lines of the file:
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@@
 <wire x1="3.81" y1="77.46" x2="3.81" y2="17.78" width="0" layer="20"/>
 <text x="6.35" y="19.05" size="1.4224" layer="21">SuperAwesomeRobots.com</text>
-<text x="19.05" y="74.93" size="1.27" layer="21" font="vector">Ultimate Voice Changer 1.1</text>
+<text x="19.05" y="74.93" size="1.4224" layer="21">Ultimate Voice Changer 1.1</text>
 <text x="31.75" y="48.26" size="1.27" layer="21" rot="R90">3.3V</text>
 <text x="29.21" y="48.26" size="1.27" layer="21" rot="R90">GND</text>
@@
 </autorouter>
 <elements>
-<element name="C1" library="SparkFun-Capacitors" package="CAP-PTH-5MM" value="0.1uF" x="38.1" y="25.4" rot="R270"/>
-<element name="C2" library="SparkFun-Capacitors" package="CPOL-RADIAL-10UF-25V" value="10uF" x="52.07" y="34.29" rot="R90"/>
-<element name="JP1" library="SparkFun-Connectors" package="AUDIO-JACK" value="" x="48.26" y="21.59" rot="R90"/>
-<element name="LED1" library="SparkFun-LED" package="LED5MM" value="" x="16.51" y="62.23" rot="R90"/>
-<element name="R1" library="SparkFun-Resistors" package="AXIAL-0.3" value="330" x="16.51" y="67.31">
+<element name="C1" library="SparkFun-Capacitors" package="CAP-PTH-5MM" value="0.1uF" x="38.1" y="25.4" smashed="yes" rot="R270">
+<attribute name="NAME" x="39.37" y="26.162" size="0.8128" layer="25" rot="R270"/>
+<attribute name="VALUE" x="35.306" y="26.416" size="0.8128" layer="27" rot="R270"/>
+</element>
+<element name="C2" library="SparkFun-Capacitors" package="CPOL-RADIAL-10UF-25V" value="10uF" x="52.07" y="34.29" smashed="yes" rot="R90">
+<attribute name="NAME" x="49.276" y="32.131" size="0.8128" layer="21" rot="R90"/>
+<attribute name="VALUE" x="55.753" y="32.385" size="0.8128" layer="27" rot="R90"/>
+</element>
+<element name="JP1" library="SparkFun-Connectors" package="AUDIO-JACK" value="" x="48.26" y="21.59" smashed="yes" rot="R90">
+<attribute name="VALUE" x="46.99" y="20.32" size="0.4064" layer="27" rot="R90"/>
+</element>
+<element name="LED" library="SparkFun-LED" package="LED5MM" value="" x="16.51" y="62.23" smashed="yes" rot="R90">
+<attribute name="NAME" x="21.0566" y="61.595" size="0.8128" layer="21" ratio="10" rot="R90"/>
+<attribute name="VALUE" x="18.3134" y="65.4304" size="1.27" layer="27" ratio="10" rot="R90"/>
+</element>
+<element name="R1" library="SparkFun-Resistors" package="AXIAL-0.3" value="330" x="16.51" y="67.31" smashed="yes">
 <attribute name="VALE" value="1k" x="16.51" y="67.31" size="1.778" layer="27" display="off"/>
 <attribute name="PROD_ID" value="RES-08380" x="16.51" y="67.31" size="1.778" layer="27" display="off"/>
-</element>
-<element name="R2" library="SparkFun-Resistors" package="AXIAL-0.3" value="1.5k" x="29.21" y="33.02">
+<attribute name="NAME" x="13.97" y="68.58" size="0.8128" layer="21" font="vector"/>
+<attribute name="VALUE" x="14.478" y="66.929" size="0.8128" layer="21" ratio="15"/>
+</element>
+<element name="R2" library="SparkFun-Resistors" package="AXIAL-0.3" value="1.5k" x="29.21" y="33.02" smashed="yes">
 <attribute name="VALE" value="1k" x="29.21" y="33.02" size="1.778" layer="27" display="off"/>
 <attribute name="PROD_ID" value="RES-08380" x="29.21" y="33.02" size="1.778" layer="27" display="off"/>
-</element>
-<element name="R3" library="SparkFun-Resistors" package="AXIAL-0.3" value="1k" x="29.21" y="29.21">
+<attribute name="NAME" x="26.67" y="34.29" size="0.8128" layer="21" font="vector"/>
+<attribute name="VALUE" x="27.178" y="32.639" size="0.8128" layer="21" ratio="15"/>
+</element>
+<element name="R3" library="SparkFun-Resistors" package="AXIAL-0.3" value="1k" x="29.21" y="29.21" smashed="yes">
 <attribute name="VALE" value="1k" x="29.21" y="29.21" size="1.778" layer="27" display="off"/>
 <attribute name="PROD_ID" value="RES-08380" x="29.21" y="29.21" size="1.778" layer="27" display="off"/>
+<attribute name="NAME" x="26.67" y="30.48" size="0.8128" layer="21" font="vector"/>
+<attribute name="VALUE" x="27.178" y="28.829" size="0.8128" layer="21" ratio="15"/>
 </element>
 <element name="U$1" library="Microchip_By_element14_Batch_1" package="DIP254P762X432-8" value="MCP4921-E/P" x="20.32" y="26.67" smashed="yes">
@@
 <attribute name="NAME" x="26.5938" y="24.6888" size="1.27" layer="25" ratio="10"/>
 </element>
-<element name="R4" library="SparkFun-Resistors" package="AXIAL-0.3" value="" x="16.51" y="22.86">
+<element name="R4" library="SparkFun-Resistors" package="AXIAL-0.3" value="" x="16.51" y="22.86" smashed="yes">
 <attribute name="VALE" value="1k" x="16.51" y="22.86" size="1.778" layer="27" display="off"/>
 <attribute name="PROD_ID" value="RES-08380" x="16.51" y="22.86" size="1.778" layer="27" display="off"/>
+<attribute name="NAME" x="13.97" y="24.13" size="0.8128" layer="21" font="vector"/>
+<attribute name="VALUE" x="14.478" y="22.479" size="1.016" layer="21" font="vector" ratio="15"/>
 </element>
 <element name="ADC2" library="SparkFun-Electromechanical" package="3386U" value="TRIMPOT-PTH-KNOB" x="43.18" y="66.04"/>
@@
 <signal name="N$1">
 <contactref element="R1" pad="P$2"/>
-<contactref element="LED1" pad="A"/>
+<contactref element="LED" pad="A"/>
 <wire x1="16.6878" y1="61.722" x2="16.6878" y2="61.0362" width="0.254" layer="1"/>
 <wire x1="20.1168" y1="65.151" x2="16.6878" y2="61.722" width="0.254" layer="1"/>
@@
 </signal>
 <signal name="GND">
-<contactref element="LED1" pad="K"/>
+<contactref element="LED" pad="K"/>
 <contactref element="U1" pad="GND@0"/>
 <contactref element="U$2" pad="7"/>

Commit message: clean up board
Parts:
- renumbered MIC to ADC1_MIC
Other:
- board text added: "ADC2"
- board text added: "ADC3"
- board text added: "ADC4"
- board text added: "AUD"
- board text removed: "ADC1"
Changed lines of the file:
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@@
 <wire x1="3.81" y1="77.46" x2="3.81" y2="17.78" width="0" layer="20"/>
 <text x="6.35" y="19.05" size="1.4224" layer="21">SuperAwesomeRobots.com</text>
-<text x="19.05" y="74.93" size="1.4224" layer="21">Ultimate Voice Changer 1.1</text>
-<text x="31.75" y="48.26" size="1.27" layer="21" rot="R90">3.3V</text>
-<text x="29.21" y="48.26" size="1.27" layer="21" rot="R90">GND</text>
-<text x="26.67" y="48.26" size="1.27" layer="21" rot="R90">ADC1</text>
+<text x="11.43" y="71.12" size="1.4224" layer="21">Ultimate Voice Changer 1.1</text>
+<text x="31.75" y="49.53" size="0.8128" layer="21" rot="R90">3.3V</text>
+<text x="29.21" y="49.53" size="0.8128" layer="21" rot="R90">GND</text>
+<text x="26.67" y="49.53" size="0.8128" layer="21" rot="R90">AUD</text>
 <text x="16.51" y="43.18" size="1.27" layer="21" rot="R90">MCP3204</text>
 <text x="15.24" y="34.29" size="1.27" layer="21" rot="SR270">MCP4921</text>
+<text x="38.1" y="71.12" size="0.8128" layer="21">ADC2</text>
+<text x="38.1" y="59.69" size="0.8128" layer="21">ADC3</text>
+<text x="38.1" y="48.26" size="0.8128" layer="21">ADC4</text>
 </plain>
 <attributes>
@@
 <element name="C1" library="SparkFun-Capacitors" package="CAP-PTH-5MM" value="0.1uF" x="38.1" y="25.4" smashed="yes" rot="R270">
 <attribute name="NAME" x="39.37" y="26.162" size="0.8128" layer="25" rot="R270"/>
-<attribute name="VALUE" x="35.306" y="26.416" size="0.8128" layer="27" rot="R270"/>
+<attribute name="VALUE" x="35.306" y="26.416" size="0.8128" layer="21" rot="R270"/>
 </element>
 <element name="C2" library="SparkFun-Capacitors" package="CPOL-RADIAL-10UF-25V" value="10uF" x="52.07" y="34.29" smashed="yes" rot="R90">
 <attribute name="NAME" x="49.276" y="32.131" size="0.8128" layer="21" rot="R90"/>
-<attribute name="VALUE" x="55.753" y="32.385" size="0.8128" layer="27" rot="R90"/>
+<attribute name="VALUE" x="55.753" y="32.385" size="0.8128" layer="21" rot="R90"/>
 </element>
 <element name="JP1" library="SparkFun-Connectors" package="AUDIO-JACK" value="" x="48.26" y="21.59" smashed="yes" rot="R90">
@@
 </element>
 <element name="U1" library="SparkFun-Boards" package="DUEMILANOVE_SHIELD" value="ARDUINO_SHIELDLABEL" x="3.81" y="17.78"/>
-<element name="MIC" library="SparkFun-Connectors" package="1X03_LOCK" value="" x="26.67" y="54.61"/>
+<element name="ADC1_MIC" library="SparkFun-Connectors" package="1X03_LOCK" value="" x="26.67" y="54.61" smashed="yes">
+<attribute name="NAME" x="25.3238" y="56.4388" size="0.8128" layer="21" ratio="10"/>
+<attribute name="VALUE" x="25.4" y="51.435" size="1.27" layer="27"/>
+</element>
 <element name="EXT_LED" library="SparkFun-Connectors" package="1X02_LOCK" value="M02LOCK" x="27.94" y="22.86" smashed="yes">
 <attribute name="NAME" x="26.5938" y="24.6888" size="1.27" layer="25" ratio="10"/>
@@
 <contactref element="R3" pad="P$1"/>
 <contactref element="JP1" pad="SLEEVE"/>
-<contactref element="MIC" pad="2"/>
+<contactref element="ADC1_MIC" pad="2"/>
 <contactref element="EXT_LED" pad="2"/>
 <contactref element="ADC2" pad="3"/>
@@
 <contactref element="U1" pad="3.3V"/>
 <contactref element="U$1" pad="6"/>
-<contactref element="MIC" pad="3"/>
+<contactref element="ADC1_MIC" pad="3"/>
 <contactref element="ADC2" pad="1"/>
 <contactref element="ADC3" pad="1"/>
@@
 <signal name="ADC1">
 <contactref element="U$2" pad="1"/>
-<contactref element="MIC" pad="1"/>
+<contactref element="ADC1_MIC" pad="1"/>
 <wire x1="20.3454" y1="40.2336" x2="20.3454" y2="39.5478" width="0.254" layer="1"/>
 <wire x1="26.5176" y1="46.4058" x2="20.3454" y2="40.2336" width="0.254" layer="1"/>

Commit message: clean up board
Other:
- board size 54.3 x 59.7 mm -> 53 x 59.7 mm
Changed lines of the file:
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@@
 <board>
 <plain>
-<wire x1="3.81" y1="17.78" x2="58.09" y2="17.78" width="0" layer="20"/>
-<wire x1="58.09" y1="17.78" x2="58.09" y2="77.46" width="0" layer="20"/>
-<wire x1="58.09" y1="77.46" x2="3.81" y2="77.46" width="0" layer="20"/>
+<wire x1="3.81" y1="17.78" x2="56.82" y2="17.78" width="0" layer="20"/>
+<wire x1="56.82" y1="17.78" x2="56.82" y2="77.46" width="0" layer="20"/>
+<wire x1="56.82" y1="77.46" x2="3.81" y2="77.46" width="0" layer="20"/>
 <wire x1="3.81" y1="77.46" x2="3.81" y2="17.78" width="0" layer="20"/>
 <text x="6.35" y="19.05" size="1.4224" layer="21">SuperAwesomeRobots.com</text>
